File: kicad/projects/FULL_BOARD_SQ5/FULL_BOARD_SQ5/sensor_matrix.kicad_sch (KiCad schematic)
At the start: 36 parts, among them U10 HALL_SENSOR_6, U11 HALL_SENSOR_10, U12 HALL_SENSOR_14, U13 HALL_SENSOR3, U14 HALL_SENSOR7, U15 HALL_SENSOR11, U16 HALL_SENSOR15, U17 HALL_SENSOR4, U18 HALL_SENSOR8, U19 HALL_SENSOR12, U20 HALL_SENSOR16, U21 CD74HC4067M, U5 HALL_SENSOR_1, U6 HALL_SENSOR_5, U7 HALL_SENSOR_9, U8 HALL_SENSOR_13, U9 HALL_SENSOR_2

Commit message: all footprints and started pcb
Parts:
- U10, U11, U12, U13, U14, U15, U16, U17, U18, U19, U20, U5, U6, U7, U8, U9: footprint Package_TO_SOT_THT:TO-92_Inline -> PCM_Package_TO_SOT_SMD_AKL:SOT-23_Handsoldering
Changed lines of the file:
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@@
 			)
 		)
-		(property "Footprint" "Package_TO_SOT_THT:TO-92_Inline"
+		(property "Footprint" "PCM_Package_TO_SOT_SMD_AKL:SOT-23_Handsoldering"
 			(at 115.57 38.1 0)
 			(effects
@@
 			)
 		)
-		(property "Footprint" "Package_TO_SOT_THT:TO-92_Inline"
+		(property "Footprint" "PCM_Package_TO_SOT_SMD_AKL:SOT-23_Handsoldering"
 			(at 115.57 80.01 0)
 			(effects
@@
 			)
 		)
-		(property "Footprint" "Package_TO_SOT_THT:TO-92_Inline"
+		(property "Footprint" "PCM_Package_TO_SOT_SMD_AKL:SOT-23_Handsoldering"
 			(at 43.18 123.19 0)
 			(effects
@@
 			)
 		)
-		(property "Footprint" "Package_TO_SOT_THT:TO-92_Inline"
+		(property "Footprint" "PCM_Package_TO_SOT_SMD_AKL:SOT-23_Handsoldering"
 			(at 151.13 38.1 0)
 			(effects
@@
 			)
 		)
-		(property "Footprint" "Package_TO_SOT_THT:TO-92_Inline"
+		(property "Footprint" "PCM_Package_TO_SOT_SMD_AKL:SOT-23_Handsoldering"
 			(at 151.13 80.01 0)
 			(effects
@@
 			)
 		)
-		(property "Footprint" "Package_TO_SOT_THT:TO-92_Inline"
+		(property "Footprint" "PCM_Package_TO_SOT_SMD_AKL:SOT-23_Handsoldering"
 			(at 151.13 123.19 0)
 			(effects
@@
 			)
 		)
-		(property "Footprint" "Package_TO_SOT_THT:TO-92_Inline"
+		(property "Footprint" "PCM_Package_TO_SOT_SMD_AKL:SOT-23_Handsoldering"
 			(at 43.18 80.01 0)
 			(effects
@@
 			)
 		)
-		(property "Footprint" "Package_TO_SOT_THT:TO-92_Inline"
+		(property "Footprint" "PCM_Package_TO_SOT_SMD_AKL:SOT-23_Handsoldering"
 			(at 80.01 165.1 0)
 			(effects
@@
 			)
 		)
-		(property "Footprint" "Package_TO_SOT_THT:TO-92_Inline"
+		(property "Footprint" "PCM_Package_TO_SOT_SMD_AKL:SOT-23_Handsoldering"
 			(at 43.18 165.1 0)
 			(effects
@@
 			)
 		)
-		(property "Footprint" "Package_TO_SOT_THT:TO-92_Inline"
+		(property "Footprint" "PCM_Package_TO_SOT_SMD_AKL:SOT-23_Handsoldering"
 			(at 151.13 165.1 0)
 			(effects
@@
 			)
 		)
-		(property "Footprint" "Package_TO_SOT_THT:TO-92_Inline"
+		(property "Footprint" "PCM_Package_TO_SOT_SMD_AKL:SOT-23_Handsoldering"
 			(at 115.57 165.1 0)
 			(effects
@@
 			)
 		)
-		(property "Footprint" "Package_TO_SOT_THT:TO-92_Inline"
+		(property "Footprint" "PCM_Package_TO_SOT_SMD_AKL:SOT-23_Handsoldering"
 			(at 43.18 38.1 0)
 			(effects
@@
 			)
 		)
-		(property "Footprint" "Package_TO_SOT_THT:TO-92_Inline"
+		(property "Footprint" "PCM_Package_TO_SOT_SMD_AKL:SOT-23_Handsoldering"
 			(at 80.01 123.19 0)
 			(effects
@@
 			)
 		)
-		(property "Footprint" "Package_TO_SOT_THT:TO-92_Inline"
+		(property "Footprint" "PCM_Package_TO_SOT_SMD_AKL:SOT-23_Handsoldering"
 			(at 115.57 123.19 0)
 			(effects
@@
 			)
 		)
-		(property "Footprint" "Package_TO_SOT_THT:TO-92_Inline"
+		(property "Footprint" "PCM_Package_TO_SOT_SMD_AKL:SOT-23_Handsoldering"
 			(at 80.01 38.1 0)
 			(effects
@@
 			)
 		)
-		(property "Footprint" "Package_TO_SOT_THT:TO-92_Inline"
+		(property "Footprint" "PCM_Package_TO_SOT_SMD_AKL:SOT-23_Handsoldering"
 			(at 80.01 80.01 0)
 			(effects
