File: kicad/projects/SENSORS_MATRIX_5CM/SENSORS_MATRIX_5CM.kicad_pcb (KiCad board)
At the start: 2 copper layers, 400 x 400 mm, 159 parts, among them J1 Conn_02x11_Odd_Even, U10 HALL_SENSOR_6, U11 HALL_SENSOR_10, U12 HALL_SENSOR_14, U13 HALL_SENSOR3, U14 HALL_SENSOR7, U15 HALL_SENSOR11, U16 HALL_SENSOR15, U17 HALL_SENSOR4, U18 HALL_SENSOR8, U19 HALL_SENSOR12, U20 HALL_SENSOR16, U21 CD74HC4067M, U22 HALL_SENSOR_1, U23 HALL_SENSOR_5, U24 HALL_SENSOR_9, U25 HALL_SENSOR_13, U26 HALL_SENSOR_2, U27 HALL_SENSOR_6, U28 HALL_SENSOR_10, U29 HALL_SENSOR_14, U30 HALL_SENSOR3, U31 HALL_SENSOR7, U32 HALL_SENSOR11, U33 HALL_SENSOR15, U34 HALL_SENSOR4, U35 HALL_SENSOR8, U36 HALL_SENSOR12, U37 HALL_SENSOR16, U38 CD74HC4067M, U39 HALL_SENSOR_1, U40 HALL_SENSOR_5, U41 HALL_SENSOR_9, U42 HALL_SENSOR_13, U43 HALL_SENSOR_2, U44 HALL_SENSOR_6, U45 HALL_SENSOR_10, U46 HALL_SENSOR_14, U47 HALL_SENSOR3, U48 HALL_SENSOR7, U49 HALL_SENSOR11, U5 HALL_SENSOR_1, U50 HALL_SENSOR15, U51 HALL_SENSOR4, U52 HALL_SENSOR8, U53 HALL_SENSOR12, U54 HALL_SENSOR16, U55 CD74HC4067M, U56 HALL_SENSOR_1, U57 HALL_SENSOR_5, U58 HALL_SENSOR_9, U59 HALL_SENSOR_13, U6 HALL_SENSOR_5, U60 HALL_SENSOR_2, U61 HALL_SENSOR_6, U62 HALL_SENSOR_10, U63 HALL_SENSOR_14, U64 HALL_SENSOR3, U65 HALL_SENSOR7, U66 HALL_SENSOR11, U67 HALL_SENSOR15, U68 HALL_SENSOR4, U69 HALL_SENSOR8, U7 HALL_SENSOR_9, U70 HALL_SENSOR12, U71 HALL_SENSOR16, U72 CD74HC4067M, U8 HALL_SENSOR_13, U9 HALL_SENSOR_2

Commit message: sensors board almost finished
Parts:
- moved R7 108.2 mm to (454.2, 193.5)
- moved D1 105.5 mm to (454.2, 191.2)
- moved R3 104.5 mm to (467.5, 211.0)
- moved R4 104.2 mm to (467.5, 213.2)
- moved R5 104.0 mm to (467.5, 215.7)
- moved R6 103.8 mm to (467.5, 218.2)
- moved D2 94.8 mm to (472.0, 211.0), turned to 0 degrees
- moved D3 94.5 mm to (472.0, 213.3), turned to 0 degrees
- moved D4 94.2 mm to (472.0, 215.8), turned to 0 degrees
- moved D5 93.9 mm to (472.0, 218.2), turned to 0 degrees
- moved R27 16.8 mm to (491.5, 195.2), turned to 180 degrees
- moved R26 15.6 mm to (491.5, 197.5), turned to 180 degrees
- moved C1 12.9 mm to (479.5, 188.0), turned to 90 degrees
- moved C2 12.1 mm to (477.2, 188.0), turned to 90 degrees
- moved C33 1.76 mm to (483.0, 155.7)
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Connections:
- J1 pad 11: SIG1 -> +3V3
- J1 pad 12: unconnected-(J1-Pin_12-Pad12) -> +3V3
- J1 pad 14: SIG2 -> FBK_3V3_SENSORS
- J1 pad 15: SIG3 -> SIG2
- J1 pad 18: SIG4 -> SIG3
- J1 pad 19: FBK_3V3_SENSORS -> SIG4
- J1 pad 2: +3V3 -> SIG1
- J1 pad 20: +3V3 -> GND
Routing:
- net +3V3: track 24.9 -> 4078.3 mm, vias 0 -> 5
- net MUX2: track 0.00 -> 420.2 mm, vias 0 -> 6
- net MUX1: track 0.00 -> 417.7 mm, vias 0 -> 6
- net MUX4: track 0.00 -> 391.4 mm, vias 0 -> 7
- net MUX3: track 0.00 -> 387.8 mm, vias 0 -> 7
- net /sensor_matrix2/hall9: track 0.00 -> 371.0 mm
- net /sensor_matrix1/hall9: track 0.00 -> 368.5 mm
- net /sensor_matrix3/hall9: track 0.00 -> 368.2 mm
- net /sensor_matrix0/hall9: track 0.00 -> 364.6 mm
- net /sensor_matrix2/hall1: track 0.00 -> 357.2 mm
- net /sensor_matrix3/hall1: track 0.00 -> 355.8 mm
- net /sensor_matrix1/hall1: track 0.00 -> 354.2 mm
- net /sensor_matrix0/hall1: track 0.00 -> 351.4 mm
- net /sensor_matrix2/hall10: track 0.00 -> 318.8 mm
- net /sensor_matrix1/hall10: track 0.00 -> 316.9 mm
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- added copper zone on F.Cu, net +3V3
- added copper zone on B.Cu, net GND
- added copper zone on F.Cu, net GND
Other:
- outline, holes or cut-outs redrawn

Commit message: brainv2
Routing:
- net +3V3: track 4078.3 -> 4128.1 mm
- net FBK_3V3_SENSORS: track 0.00 -> 8.16 mm

Commit message: brain v2, all components placed?
Parts:
- R16, R17, R18, R19: value 10K -> 10k

Commit message: hw revisions and versions in schematic and pins
Parts:
- removed R26: 10k, Resistor_SMD:R_0805_2012Metric_Pad1.20x1.40mm_HandSolder
- removed R27: 100k, Resistor_SMD:R_0805_2012Metric_Pad1.20x1.40mm_HandSolder
- added R1: 0, Resistor_SMD:R_0805_2012Metric_Pad1.20x1.40mm_HandSolder, B.Cu at (482.8, 176.2)
- added R13: 0, Resistor_SMD:R_0805_2012Metric_Pad1.20x1.40mm_HandSolder, B.Cu at (482.8, 174.2)
- added R2: 0, Resistor_SMD:R_0805_2012Metric_Pad1.20x1.40mm_HandSolder, B.Cu at (482.8, 180.5)
- added R8: 0, Resistor_SMD:R_0805_2012Metric_Pad1.20x1.40mm_HandSolder, B.Cu at (482.8, 182.5)
- added R9: 0, Resistor_SMD:R_0805_2012Metric_Pad1.20x1.40mm_HandSolder, B.Cu at (482.8, 184.8)
- moved J1 9.61 mm to (487.0, 174.3)
Connections:
- C1 pad 1: +3V3 -> FBK_3V3_SENSORS
- C17 pad 1: +3V3 -> FBK_3V3_SENSORS
- C18 pad 1: +3V3 -> FBK_3V3_SENSORS
- C19 pad 1: +3V3 -> FBK_3V3_SENSORS
- C2 pad 1: +3V3 -> FBK_3V3_SENSORS
- C20 pad 1: +3V3 -> FBK_3V3_SENSORS
- C21 pad 1: +3V3 -> FBK_3V3_SENSORS
- C22 pad 1: +3V3 -> FBK_3V3_SENSORS
- C23 pad 1: +3V3 -> FBK_3V3_SENSORS
- C24 pad 1: +3V3 -> FBK_3V3_SENSORS
- C25 pad 1: +3V3 -> FBK_3V3_SENSORS
- C26 pad 1: +3V3 -> FBK_3V3_SENSORS
- C27 pad 1: +3V3 -> FBK_3V3_SENSORS
- C28 pad 1: +3V3 -> FBK_3V3_SENSORS
- C29 pad 1: +3V3 -> FBK_3V3_SENSORS
- C30 pad 1: +3V3 -> FBK_3V3_SENSORS
- C31 pad 1: +3V3 -> FBK_3V3_SENSORS
- C32 pad 1: +3V3 -> FBK_3V3_SENSORS
- C33 pad 1: +3V3 -> FBK_3V3_SENSORS
- C34 pad 1: +3V3 -> FBK_3V3_SENSORS
- C35 pad 1: +3V3 -> FBK_3V3_SENSORS
- C36 pad 1: +3V3 -> FBK_3V3_SENSORS
- C37 pad 1: +3V3 -> FBK_3V3_SENSORS
- C38 pad 1: +3V3 -> FBK_3V3_SENSORS
- C39 pad 1: +3V3 -> FBK_3V3_SENSORS
- C40 pad 1: +3V3 -> FBK_3V3_SENSORS
- C41 pad 1: +3V3 -> FBK_3V3_SENSORS
- C42 pad 1: +3V3 -> FBK_3V3_SENSORS
- C43 pad 1: +3V3 -> FBK_3V3_SENSORS
- C44 pad 1: +3V3 -> FBK_3V3_SENSORS
- C45 pad 1: +3V3 -> FBK_3V3_SENSORS
- C46 pad 1: +3V3 -> FBK_3V3_SENSORS
- C47 pad 1: +3V3 -> FBK_3V3_SENSORS
- C48 pad 1: +3V3 -> FBK_3V3_SENSORS
- C49 pad 1: +3V3 -> FBK_3V3_SENSORS
- C50 pad 1: +3V3 -> FBK_3V3_SENSORS
- C51 pad 1: +3V3 -> FBK_3V3_SENSORS
- C52 pad 1: +3V3 -> FBK_3V3_SENSORS
- C53 pad 1: +3V3 -> FBK_3V3_SENSORS
- C54 pad 1: +3V3 -> FBK_3V3_SENSORS
- C55 pad 1: +3V3 -> FBK_3V3_SENSORS
- C56 pad 1: +3V3 -> FBK_3V3_SENSORS
- C57 pad 1: +3V3 -> FBK_3V3_SENSORS
- C58 pad 1: +3V3 -> FBK_3V3_SENSORS
- C59 pad 1: +3V3 -> FBK_3V3_SENSORS
- C60 pad 1: +3V3 -> FBK_3V3_SENSORS
- C61 pad 1: +3V3 -> FBK_3V3_SENSORS
- C62 pad 1: +3V3 -> FBK_3V3_SENSORS
- C63 pad 1: +3V3 -> FBK_3V3_SENSORS
- C64 pad 1: +3V3 -> FBK_3V3_SENSORS
- C65 pad 1: +3V3 -> FBK_3V3_SENSORS
- C66 pad 1: +3V3 -> FBK_3V3_SENSORS
- C67 pad 1: +3V3 -> FBK_3V3_SENSORS
- C68 pad 1: +3V3 -> FBK_3V3_SENSORS
- C69 pad 1: +3V3 -> FBK_3V3_SENSORS
- C70 pad 1: +3V3 -> FBK_3V3_SENSORS
- C71 pad 1: +3V3 -> FBK_3V3_SENSORS
- C72 pad 1: +3V3 -> FBK_3V3_SENSORS
- C73 pad 1: +3V3 -> FBK_3V3_SENSORS
- C74 pad 1: +3V3 -> FBK_3V3_SENSORS
- C75 pad 1: +3V3 -> FBK_3V3_SENSORS
- C76 pad 1: +3V3 -> FBK_3V3_SENSORS
- C77 pad 1: +3V3 -> FBK_3V3_SENSORS
- C78 pad 1: +3V3 -> FBK_3V3_SENSORS
- C79 pad 1: +3V3 -> FBK_3V3_SENSORS
- C80 pad 1: +3V3 -> FBK_3V3_SENSORS
- C81 pad 1: +3V3 -> FBK_3V3_SENSORS
- C82 pad 1: +3V3 -> FBK_3V3_SENSORS
- C83 pad 1: +3V3 -> FBK_3V3_SENSORS
- C84 pad 1: +3V3 -> FBK_3V3_SENSORS
- C85 pad 1: +3V3 -> FBK_3V3_SENSORS
- C86 pad 1: +3V3 -> FBK_3V3_SENSORS
- C87 pad 1: +3V3 -> FBK_3V3_SENSORS
- C88 pad 1: +3V3 -> FBK_3V3_SENSORS
- D1 pad 2: +3V3 -> FBK_3V3_SENSORS
- J1 pad 10: MUX4 -> MUX2
- J1 pad 11: +3V3 -> MUX3
- J1 pad 12: +3V3 -> MUX4
- J1 pad 13: GND -> FBK_3V3_SENSORS
- J1 pad 15: SIG2 -> GND
- J1 pad 16: GND -> FBK_3V3_SENSORS
- J1 pad 17: GND -> SIG2
- J1 pad 18: SIG3 -> GND
- J1 pad 19: SIG4 -> GND
- J1 pad 20: GND -> SIG3
- J1 pad 21: GND -> SIG4
- J1 pad 3: MUX1 -> PCB_REV0
- J1 pad 4: GND -> PCB_REV1
- J1 pad 5: GND -> HW_ID0
- J1 pad 6: MUX2 -> HW_ID1
- J1 pad 7: MUX3 -> FBK_3V3_SENSORS
- J1 pad 8: GND -> HW_ID2
- J1 pad 9: +3V3 -> MUX1
- U10 pad 1: +3V3 -> FBK_3V3_SENSORS
- U11 pad 1: +3V3 -> FBK_3V3_SENSORS
- U12 pad 1: +3V3 -> FBK_3V3_SENSORS
- U13 pad 1: +3V3 -> FBK_3V3_SENSORS
- U14 pad 1: +3V3 -> FBK_3V3_SENSORS
- U15 pad 1: +3V3 -> FBK_3V3_SENSORS
- U16 pad 1: +3V3 -> FBK_3V3_SENSORS
- U17 pad 1: +3V3 -> FBK_3V3_SENSORS
- U18 pad 1: +3V3 -> FBK_3V3_SENSORS
- U19 pad 1: +3V3 -> FBK_3V3_SENSORS
- U20 pad 1: +3V3 -> FBK_3V3_SENSORS
- U21 pad 24: +3V3 -> FBK_3V3_SENSORS
- U22 pad 1: +3V3 -> FBK_3V3_SENSORS
- U23 pad 1: +3V3 -> FBK_3V3_SENSORS
- U24 pad 1: +3V3 -> FBK_3V3_SENSORS
- U25 pad 1: +3V3 -> FBK_3V3_SENSORS
- U26 pad 1: +3V3 -> FBK_3V3_SENSORS
- U27 pad 1: +3V3 -> FBK_3V3_SENSORS
- U28 pad 1: +3V3 -> FBK_3V3_SENSORS
- U29 pad 1: +3V3 -> FBK_3V3_SENSORS
- U30 pad 1: +3V3 -> FBK_3V3_SENSORS
- U31 pad 1: +3V3 -> FBK_3V3_SENSORS
- U32 pad 1: +3V3 -> FBK_3V3_SENSORS
- U33 pad 1: +3V3 -> FBK_3V3_SENSORS
- U34 pad 1: +3V3 -> FBK_3V3_SENSORS
- U35 pad 1: +3V3 -> FBK_3V3_SENSORS
- U36 pad 1: +3V3 -> FBK_3V3_SENSORS
- U37 pad 1: +3V3 -> FBK_3V3_SENSORS
- U38 pad 24: +3V3 -> FBK_3V3_SENSORS
- U39 pad 1: +3V3 -> FBK_3V3_SENSORS
- U40 pad 1: +3V3 -> FBK_3V3_SENSORS
- U41 pad 1: +3V3 -> FBK_3V3_SENSORS
- U42 pad 1: +3V3 -> FBK_3V3_SENSORS
- U43 pad 1: +3V3 -> FBK_3V3_SENSORS
- U44 pad 1: +3V3 -> FBK_3V3_SENSORS
- U45 pad 1: +3V3 -> FBK_3V3_SENSORS
- U46 pad 1: +3V3 -> FBK_3V3_SENSORS
- U47 pad 1: +3V3 -> FBK_3V3_SENSORS
- U48 pad 1: +3V3 -> FBK_3V3_SENSORS
- U49 pad 1: +3V3 -> FBK_3V3_SENSORS
- U5 pad 1: +3V3 -> FBK_3V3_SENSORS
- U50 pad 1: +3V3 -> FBK_3V3_SENSORS
- U51 pad 1: +3V3 -> FBK_3V3_SENSORS
- U52 pad 1: +3V3 -> FBK_3V3_SENSORS
- U53 pad 1: +3V3 -> FBK_3V3_SENSORS
- U54 pad 1: +3V3 -> FBK_3V3_SENSORS
- U55 pad 24: +3V3 -> FBK_3V3_SENSORS
- U56 pad 1: +3V3 -> FBK_3V3_SENSORS
- U57 pad 1: +3V3 -> FBK_3V3_SENSORS
- U58 pad 1: +3V3 -> FBK_3V3_SENSORS
- U59 pad 1: +3V3 -> FBK_3V3_SENSORS
- U6 pad 1: +3V3 -> FBK_3V3_SENSORS
- U60 pad 1: +3V3 -> FBK_3V3_SENSORS
- U61 pad 1: +3V3 -> FBK_3V3_SENSORS
- U62 pad 1: +3V3 -> FBK_3V3_SENSORS
- U63 pad 1: +3V3 -> FBK_3V3_SENSORS
- U64 pad 1: +3V3 -> FBK_3V3_SENSORS
- U65 pad 1: +3V3 -> FBK_3V3_SENSORS
- U66 pad 1: +3V3 -> FBK_3V3_SENSORS
- U67 pad 1: +3V3 -> FBK_3V3_SENSORS
- U68 pad 1: +3V3 -> FBK_3V3_SENSORS
- U69 pad 1: +3V3 -> FBK_3V3_SENSORS
- U7 pad 1: +3V3 -> FBK_3V3_SENSORS
- U70 pad 1: +3V3 -> FBK_3V3_SENSORS
- U71 pad 1: +3V3 -> FBK_3V3_SENSORS
- U72 pad 24: +3V3 -> FBK_3V3_SENSORS
- U8 pad 1: +3V3 -> FBK_3V3_SENSORS
- U9 pad 1: +3V3 -> FBK_3V3_SENSORS
Routing:
- net +3V3: track 4128.1 -> 0.00 mm, vias 5 -> 0
- net FBK_3V3_SENSORS: track 8.16 -> 4034.5 mm, vias 0 -> 7
- net SIG1: track 42.5 -> 34.9 mm
- net MUX4: track 391.4 -> 398.4 mm
- net HW_ID1: track 0.00 -> 7.02 mm
- net PCB_REV1: track 0.00 -> 6.97 mm
- net HW_ID2: track 0.00 -> 6.90 mm
- net MUX1: track 417.7 -> 411.2 mm
- net SIG4: track 249.2 -> 253.5 mm
- net PCB_REV0: track 0.00 -> 4.30 mm
- net MUX2: track 420.0 -> 415.9 mm, vias 6 -> 8
- net HW_ID0: track 0.00 -> 3.65 mm
- net SIG3: track 152.5 -> 155.7 mm
- net SIG2: track 52.0 -> 51.2 mm
- added copper zone on F.Cu, net FBK_3V3_SENSORS
- removed copper zone on F.Cu, net +3V3

Commit message: small adjustments
Parts:
- added R10: 0, Resistor_SMD:R_0805_2012Metric_Pad1.20x1.40mm_HandSolder, F.Cu at (492.5, 191.0)
Connections:
- C1 pad 1: FBK_3V3_SENSORS -> +3V3
- C17 pad 1: FBK_3V3_SENSORS -> +3V3
- C18 pad 1: FBK_3V3_SENSORS -> +3V3
- C19 pad 1: FBK_3V3_SENSORS -> +3V3
- C2 pad 1: FBK_3V3_SENSORS -> +3V3
- C20 pad 1: FBK_3V3_SENSORS -> +3V3
- C21 pad 1: FBK_3V3_SENSORS -> +3V3
- C22 pad 1: FBK_3V3_SENSORS -> +3V3
- C23 pad 1: FBK_3V3_SENSORS -> +3V3
- C24 pad 1: FBK_3V3_SENSORS -> +3V3
- C25 pad 1: FBK_3V3_SENSORS -> +3V3
- C26 pad 1: FBK_3V3_SENSORS -> +3V3
- C27 pad 1: FBK_3V3_SENSORS -> +3V3
- C28 pad 1: FBK_3V3_SENSORS -> +3V3
- C29 pad 1: FBK_3V3_SENSORS -> +3V3
- C30 pad 1: FBK_3V3_SENSORS -> +3V3
- C31 pad 1: FBK_3V3_SENSORS -> +3V3
- C32 pad 1: FBK_3V3_SENSORS -> +3V3
- C33 pad 1: FBK_3V3_SENSORS -> +3V3
- C34 pad 1: FBK_3V3_SENSORS -> +3V3
- C35 pad 1: FBK_3V3_SENSORS -> +3V3
- C36 pad 1: FBK_3V3_SENSORS -> +3V3
- C37 pad 1: FBK_3V3_SENSORS -> +3V3
- C38 pad 1: FBK_3V3_SENSORS -> +3V3
- C39 pad 1: FBK_3V3_SENSORS -> +3V3
- C40 pad 1: FBK_3V3_SENSORS -> +3V3
- C41 pad 1: FBK_3V3_SENSORS -> +3V3
- C42 pad 1: FBK_3V3_SENSORS -> +3V3
- C43 pad 1: FBK_3V3_SENSORS -> +3V3
- C44 pad 1: FBK_3V3_SENSORS -> +3V3
- C45 pad 1: FBK_3V3_SENSORS -> +3V3
- C46 pad 1: FBK_3V3_SENSORS -> +3V3
- C47 pad 1: FBK_3V3_SENSORS -> +3V3
- C48 pad 1: FBK_3V3_SENSORS -> +3V3
- C49 pad 1: FBK_3V3_SENSORS -> +3V3
- C50 pad 1: FBK_3V3_SENSORS -> +3V3
- C51 pad 1: FBK_3V3_SENSORS -> +3V3
- C52 pad 1: FBK_3V3_SENSORS -> +3V3
- C53 pad 1: FBK_3V3_SENSORS -> +3V3
- C54 pad 1: FBK_3V3_SENSORS -> +3V3
- C55 pad 1: FBK_3V3_SENSORS -> +3V3
- C56 pad 1: FBK_3V3_SENSORS -> +3V3
- C57 pad 1: FBK_3V3_SENSORS -> +3V3
- C58 pad 1: FBK_3V3_SENSORS -> +3V3
- C59 pad 1: FBK_3V3_SENSORS -> +3V3
- C60 pad 1: FBK_3V3_SENSORS -> +3V3
- C61 pad 1: FBK_3V3_SENSORS -> +3V3
- C62 pad 1: FBK_3V3_SENSORS -> +3V3
- C63 pad 1: FBK_3V3_SENSORS -> +3V3
- C64 pad 1: FBK_3V3_SENSORS -> +3V3
- C65 pad 1: FBK_3V3_SENSORS -> +3V3
- C66 pad 1: FBK_3V3_SENSORS -> +3V3
- C67 pad 1: FBK_3V3_SENSORS -> +3V3
- C68 pad 1: FBK_3V3_SENSORS -> +3V3
- C69 pad 1: FBK_3V3_SENSORS -> +3V3
- C70 pad 1: FBK_3V3_SENSORS -> +3V3
- C71 pad 1: FBK_3V3_SENSORS -> +3V3
- C72 pad 1: FBK_3V3_SENSORS -> +3V3
- C73 pad 1: FBK_3V3_SENSORS -> +3V3
- C74 pad 1: FBK_3V3_SENSORS -> +3V3
- C75 pad 1: FBK_3V3_SENSORS -> +3V3
- C76 pad 1: FBK_3V3_SENSORS -> +3V3
- C77 pad 1: FBK_3V3_SENSORS -> +3V3
- C78 pad 1: FBK_3V3_SENSORS -> +3V3
- C79 pad 1: FBK_3V3_SENSORS -> +3V3
- C80 pad 1: FBK_3V3_SENSORS -> +3V3
- C81 pad 1: FBK_3V3_SENSORS -> +3V3
- C82 pad 1: FBK_3V3_SENSORS -> +3V3
- C83 pad 1: FBK_3V3_SENSORS -> +3V3
- C84 pad 1: FBK_3V3_SENSORS -> +3V3
- C85 pad 1: FBK_3V3_SENSORS -> +3V3
- C86 pad 1: FBK_3V3_SENSORS -> +3V3
- C87 pad 1: FBK_3V3_SENSORS -> +3V3
- C88 pad 1: FBK_3V3_SENSORS -> +3V3
- D1 pad 2: FBK_3V3_SENSORS -> +3V3
- J1 pad 13: FBK_3V3_SENSORS -> +3V3
- J1 pad 14: FBK_3V3_SENSORS -> +3V3
- J1 pad 7: FBK_3V3_SENSORS -> +3V3
- U10 pad 1: FBK_3V3_SENSORS -> +3V3
- U11 pad 1: FBK_3V3_SENSORS -> +3V3
- U12 pad 1: FBK_3V3_SENSORS -> +3V3
- U13 pad 1: FBK_3V3_SENSORS -> +3V3
- U14 pad 1: FBK_3V3_SENSORS -> +3V3
- U15 pad 1: FBK_3V3_SENSORS -> +3V3
- U16 pad 1: FBK_3V3_SENSORS -> +3V3
- U17 pad 1: FBK_3V3_SENSORS -> +3V3
- U18 pad 1: FBK_3V3_SENSORS -> +3V3
- U19 pad 1: FBK_3V3_SENSORS -> +3V3
- U20 pad 1: FBK_3V3_SENSORS -> +3V3
- U21 pad 24: FBK_3V3_SENSORS -> +3V3
- U22 pad 1: FBK_3V3_SENSORS -> +3V3
- U23 pad 1: FBK_3V3_SENSORS -> +3V3
- U24 pad 1: FBK_3V3_SENSORS -> +3V3
- U25 pad 1: FBK_3V3_SENSORS -> +3V3
- U26 pad 1: FBK_3V3_SENSORS -> +3V3
- U27 pad 1: FBK_3V3_SENSORS -> +3V3
- U28 pad 1: FBK_3V3_SENSORS -> +3V3
- U29 pad 1: FBK_3V3_SENSORS -> +3V3
- U30 pad 1: FBK_3V3_SENSORS -> +3V3
- U31 pad 1: FBK_3V3_SENSORS -> +3V3
- U32 pad 1: FBK_3V3_SENSORS -> +3V3
- U33 pad 1: FBK_3V3_SENSORS -> +3V3
- U34 pad 1: FBK_3V3_SENSORS -> +3V3
- U35 pad 1: FBK_3V3_SENSORS -> +3V3
- U36 pad 1: FBK_3V3_SENSORS -> +3V3
- U37 pad 1: FBK_3V3_SENSORS -> +3V3
- U38 pad 24: FBK_3V3_SENSORS -> +3V3
- U39 pad 1: FBK_3V3_SENSORS -> +3V3
- U40 pad 1: FBK_3V3_SENSORS -> +3V3
- U41 pad 1: FBK_3V3_SENSORS -> +3V3
- U42 pad 1: FBK_3V3_SENSORS -> +3V3
- U43 pad 1: FBK_3V3_SENSORS -> +3V3
- U44 pad 1: FBK_3V3_SENSORS -> +3V3
- U45 pad 1: FBK_3V3_SENSORS -> +3V3
- U46 pad 1: FBK_3V3_SENSORS -> +3V3
- U47 pad 1: FBK_3V3_SENSORS -> +3V3
- U48 pad 1: FBK_3V3_SENSORS -> +3V3
- U49 pad 1: FBK_3V3_SENSORS -> +3V3
- U5 pad 1: FBK_3V3_SENSORS -> +3V3
- U50 pad 1: FBK_3V3_SENSORS -> +3V3
- U51 pad 1: FBK_3V3_SENSORS -> +3V3
- U52 pad 1: FBK_3V3_SENSORS -> +3V3
- U53 pad 1: FBK_3V3_SENSORS -> +3V3
- U54 pad 1: FBK_3V3_SENSORS -> +3V3
- U55 pad 24: FBK_3V3_SENSORS -> +3V3
- U56 pad 1: FBK_3V3_SENSORS -> +3V3
- U57 pad 1: FBK_3V3_SENSORS -> +3V3
- U58 pad 1: FBK_3V3_SENSORS -> +3V3
- U59 pad 1: FBK_3V3_SENSORS -> +3V3
- U6 pad 1: FBK_3V3_SENSORS -> +3V3
- U60 pad 1: FBK_3V3_SENSORS -> +3V3
- U61 pad 1: FBK_3V3_SENSORS -> +3V3
- U62 pad 1: FBK_3V3_SENSORS -> +3V3
- U63 pad 1: FBK_3V3_SENSORS -> +3V3
- U64 pad 1: FBK_3V3_SENSORS -> +3V3
- U65 pad 1: FBK_3V3_SENSORS -> +3V3
- U66 pad 1: FBK_3V3_SENSORS -> +3V3
- U67 pad 1: FBK_3V3_SENSORS -> +3V3
- U68 pad 1: FBK_3V3_SENSORS -> +3V3
- U69 pad 1: FBK_3V3_SENSORS -> +3V3
- U7 pad 1: FBK_3V3_SENSORS -> +3V3
- U70 pad 1: FBK_3V3_SENSORS -> +3V3
- U71 pad 1: FBK_3V3_SENSORS -> +3V3
- U72 pad 24: FBK_3V3_SENSORS -> +3V3
- U8 pad 1: FBK_3V3_SENSORS -> +3V3
- U9 pad 1: FBK_3V3_SENSORS -> +3V3
Routing:
- net +3V3: track 0.00 -> 4034.1 mm, vias 0 -> 7
- net FBK_3V3_SENSORS: track 4034.5 -> 3.05 mm, vias 7 -> 0

Commit message: sensors matrix with jlcpcb
Parts:
- C2: footprint Capacitor_SMD:C_0805_2012Metric_Pad1.18x1.45mm_HandSolder -> Capacitor_SMD:C_1206_3216Metric_Pad1.33x1.80mm_HandSolder
- U10, U27, U44, U61: value HALL_SENSOR_6 -> DRV5055Z4QDBZR
- U11, U28, U45, U62: value HALL_SENSOR_10 -> DRV5055Z4QDBZR
- U12, U29, U46, U63: value HALL_SENSOR_14 -> DRV5055Z4QDBZR
- U13, U30, U47, U64: value HALL_SENSOR3 -> DRV5055Z4QDBZR
- U14, U31, U48, U65: value HALL_SENSOR7 -> DRV5055Z4QDBZR
- U15, U32, U49, U66: value HALL_SENSOR11 -> DRV5055Z4QDBZR
- U16, U33, U50, U67: value HALL_SENSOR15 -> DRV5055Z4QDBZR
- U17, U34, U51, U68: value HALL_SENSOR4 -> DRV5055Z4QDBZR
- U18, U35, U52, U69: value HALL_SENSOR8 -> DRV5055Z4QDBZR
- U19, U36, U53, U70: value HALL_SENSOR12 -> DRV5055Z4QDBZR
- U20, U37, U54, U71: value HALL_SENSOR16 -> DRV5055Z4QDBZR
- U22, U39, U5, U56: value HALL_SENSOR_1 -> DRV5055Z4QDBZR
- U23, U40, U57, U6: value HALL_SENSOR_5 -> DRV5055Z4QDBZR
- U24, U41, U58, U7: value HALL_SENSOR_9 -> DRV5055Z4QDBZR
- U25, U42, U59, U8: value HALL_SENSOR_13 -> DRV5055Z4QDBZR
- U26, U43, U60, U9: value HALL_SENSOR_2 -> DRV5055Z4QDBZR
- moved C2 0.40 mm to (477.0, 187.7)
