File: kicad/projects/SENSORS_MATRIX_5CM/sensor_matrix.kicad_sch (KiCad schematic)
At the start: 36 parts, among them U10 HALL_SENSOR_6, U11 HALL_SENSOR_10, U12 HALL_SENSOR_14, U13 HALL_SENSOR3, U14 HALL_SENSOR7, U15 HALL_SENSOR11, U16 HALL_SENSOR15, U17 HALL_SENSOR4, U18 HALL_SENSOR8, U19 HALL_SENSOR12, U20 HALL_SENSOR16, U21 CD74HC4067M, U5 HALL_SENSOR_1, U6 HALL_SENSOR_5, U7 HALL_SENSOR_9, U8 HALL_SENSOR_13, U9 HALL_SENSOR_2

Commit message: sensors board almost finished
Parts:
- C33: LCSC p/n (none) -> C24123; MP (none) -> CL21A105KOFNNNE; shop (none) -> https://www.lcsc.com/product-detail/Multilayer-Ceramic-Capa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
- R16: value 10K -> 10k; LCSC p/n (none) -> C84376; MP (none) -> RC0805FR-0710KL; shop (none) -> https://www.lcsc.com/product-detail/Chip-Resistor-Surface-M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
- U10, U11, U12, U13, U14, U15, U16, U17, U18, U19, U20, U5, U6, U7, U8, U9: LCSC p/n (none) -> C2864477; MP (none) -> DRV5055Z4QDBZR; shop (none) -> https://www.lcsc.com/product-detail/C2864477.html
- U21: LCSC p/n (none) -> C496123; MP (none) -> CD74HC4067M96; shop (none) -> https://www.lcsc.com/product-detail/C496123.html?s_z=s_p_CD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

Commit message: sensors matrix with jlcpcb
Parts:
- C17, C18, C19, C20, C21, C22, C23, C24, C25, C26, C27, C28, C29, C30, C31, C32, C34: LCSC p/n (none) -> C1711; MP (none) -> CL21B104KBCNNNC; shop (none) -> https://www.lcsc.com/product-detail/Multilayer-Ceramic-Capa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
- U10: value HALL_SENSOR_6 -> DRV5055Z4QDBZR
- U11: value HALL_SENSOR_10 -> DRV5055Z4QDBZR
- U12: value HALL_SENSOR_14 -> DRV5055Z4QDBZR
- U13: value HALL_SENSOR3 -> DRV5055Z4QDBZR
- U14: value HALL_SENSOR7 -> DRV5055Z4QDBZR
- U15: value HALL_SENSOR11 -> DRV5055Z4QDBZR
- U16: value HALL_SENSOR15 -> DRV5055Z4QDBZR
- U17: value HALL_SENSOR4 -> DRV5055Z4QDBZR
- U18: value HALL_SENSOR8 -> DRV5055Z4QDBZR
- U19: value HALL_SENSOR12 -> DRV5055Z4QDBZR
- U20: value HALL_SENSOR16 -> DRV5055Z4QDBZR
- U5: value HALL_SENSOR_1 -> DRV5055Z4QDBZR
- U6: value HALL_SENSOR_5 -> DRV5055Z4QDBZR
- U7: value HALL_SENSOR_9 -> DRV5055Z4QDBZR
- U8: value HALL_SENSOR_13 -> DRV5055Z4QDBZR
- U9: value HALL_SENSOR_2 -> DRV5055Z4QDBZR
