File: kicad/projects/chessboard_5cm/interconnect/interconnect.kicad_pcb (KiCad board)
At the start: 2 copper layers, 40 x 380 mm, 7 parts, among them J1 PZ254-1-13-W-8.5, J10 PM254-1-08-W-8.5, J11 PM254-1-08-W-8.5, J6 PM254-1-08-W-8.5, J8 PM254-1-08-W-8.5

Commit message: brain completed
Parts:
- moved J1 25.0 mm to (85.2, 400.8)
- moved C1 22.5 mm to (84.1, 397.2)
- moved C22 22.5 mm to (84.1, 394.8)
Routing:
- net MUX3: track 378.1 -> 353.0 mm
- net MUX4: track 373.1 -> 348.1 mm
- net SIG2: track 269.4 -> 244.4 mm
- net SIG4: track 67.3 -> 42.3 mm
- net SIG3: track 168.3 -> 143.3 mm
- net SIG1: track 370.4 -> 345.4 mm
- net MUX2: track 381.9 -> 356.9 mm
- net MUX1: track 387.1 -> 362.1 mm
- net +3V3: track 422.3 -> 403.2 mm
- net GND: vias 202 -> 174
Other:
- board size 40 x 380 mm -> 40 x 355 mm
