File: kicad/projects/chessboard_5cm/SENSORS_2ROW_5CM/SENSORS_2ROW_5CM.kicad_pcb (KiCad board)
At the start: 2 copper layers, 400 x 100 mm, 49 parts, among them J2 Conn_02x05_Odd_Even, U1 DRV5055Z4QDBZR, U10 DRV5055Z4QDBZR, U11 DRV5055Z4QDBZR, U12 DRV5055Z4QDBZR, U13 DRV5055Z4QDBZR, U14 DRV5055Z4QDBZR, U15 DRV5055Z4QDBZR, U16 DRV5055Z4QDBZR, U17 CD74HC4067M, U2 DRV5055Z4QDBZR, U3 DRV5055Z4QDBZR, U4 DRV5055Z4QDBZR, U5 DRV5055Z4QDBZR, U6 DRV5055Z4QDBZR, U7 DRV5055Z4QDBZR, U8 DRV5055Z4QDBZR, U9 DRV5055Z4QDBZR

Commit message: finishing 2row 5cm pcb
Parts:
- removed R6: 220Ω, Resistor_SMD:R_0805_2012Metric_Pad1.20x1.40mm_HandSolder
- added R2: 5.1k, Resistor_SMD:R_0805_2012Metric_Pad1.20x1.40mm_HandSolder, B.Cu at (480.5, 154.0)
- D1, D2, D3, D4, D5, J2, R7: moved to B.Cu
- R3, R4, R5: value 220Ω -> 5.1k; moved to B.Cu
- moved U14 316.3 mm to (475.0, 125.0)
- moved U16 306.7 mm to (475.0, 175.0)
- moved U10 275.1 mm to (425.0, 125.0)
- moved U12 264.1 mm to (425.0, 175.0)
- moved C14 247.1 mm to (470.0, 125.0), turned to -90 degrees
- moved U6 234.7 mm to (375.0, 125.0)
- moved J2 233.3 mm to (495.0, 150.0), turned to 180 degrees
- moved C17 231.4 mm to (474.0, 157.5), turned to -90 degrees
- moved C20 231.2 mm to (493.5, 164.0), turned to 180 degrees
- moved C18 230.0 mm to (471.8, 157.5), turned to -90 degrees
- moved C16 223.1 mm to (470.0, 175.0), turned to -90 degrees
- moved U8 221.7 mm to (375.0, 175.0)
- moved C19 220.0 mm to (494.1, 167.0), turned to 180 degrees
- moved D5 216.4 mm to (484.5, 160.8)
- moved D4 216.1 mm to (484.5, 158.5)
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Connections:
- R3 pad 1: Net-(D2-K) -> Net-(D3-K)
- R4 pad 1: Net-(D3-K) -> Net-(D4-K)
- R5 pad 1: Net-(D4-K) -> Net-(D5-K)
Routing:
- net +3V3: track 0.00 -> 954.8 mm, vias 0 -> 1
- net /sensor_matrix0/hall9: track 0.00 -> 354.9 mm
- net /sensor_matrix0/hall1: track 0.00 -> 342.3 mm
- net /sensor_matrix0/hall10: track 0.00 -> 303.0 mm
- net /sensor_matrix0/hall2: track 0.00 -> 293.5 mm
- net /sensor_matrix0/hall11: track 0.00 -> 251.4 mm
- net /sensor_matrix0/hall3: track 0.00 -> 245.2 mm
- net /sensor_matrix0/hall12: track 0.00 -> 200.1 mm
- net /sensor_matrix0/hall4: track 0.00 -> 196.4 mm
- net /sensor_matrix0/hall13: track 0.00 -> 148.4 mm
- net /sensor_matrix0/hall5: track 0.00 -> 147.7 mm
- net /sensor_matrix0/hall6: track 0.00 -> 99.0 mm
- net /sensor_matrix0/hall14: track 0.00 -> 96.8 mm
- net MUX3: track 0.00 -> 57.2 mm
- net MUX4: track 0.00 -> 51.9 mm
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- added copper zone on B.Cu, net GND
- added copper zone on F.Cu, net GND
Other:
- board size 400 x 100 mm -> 400 x 99 mm

Commit message: two rows optimized
Routing:
- net GND: vias 94 -> 65
Other:
- board size 400 x 99 mm -> 400 x 60 mm

Commit message: interconnect 5cm finished. brain v2 with changes pending
Parts:
- removed C19: 1uF, Capacitor_SMD:C_0805_2012Metric_Pad1.18x1.45mm_HandSolder
- removed C20: 22uF, Capacitor_SMD:C_1206_3216Metric_Pad1.33x1.80mm_HandSolder
- removed J2: Conn_02x05_Odd_Even, Connector_PinHeader_2.54mm:PinHeader_2x05_P2.54mm_Vertical
- added C21: 1uF, Capacitor_SMD:C_0805_2012Metric_Pad1.18x1.45mm_HandSolder, F.Cu at (493.2, 159.0)
- added C22: 22uF, Capacitor_SMD:C_1206_3216Metric_Pad1.33x1.80mm_HandSolder, F.Cu at (492.8, 161.2)
- added J1: Conn_01x08, Connector_PinHeader_2.54mm:PinHeader_1x08_P2.54mm_Horizontal, B.Cu at (495.8, 155.8)
Routing:
- net +3V3: track 954.8 -> 973.7 mm
- net MUX1: track 50.5 -> 41.2 mm
- net MUX4: track 51.9 -> 59.2 mm
- net MUX2: track 48.1 -> 41.7 mm
- net SIG1: track 24.2 -> 29.6 mm
- net MUX3: track 57.2 -> 62.0 mm
- net GND: vias 65 -> 64

Commit message: brain completed
Routing:
- net MUX1: track 41.2 -> 56.3 mm
- net MUX2: track 41.7 -> 56.6 mm
- net +3V3: track 973.7 -> 962.5 mm
- net MUX3: track 62.0 -> 52.3 mm
- net MUX4: track 59.2 -> 52.0 mm
Changed lines of the file:
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@@
-	)
-	(segment
-		(start 490.91 164.25)
-		(end 495 160.16)
-		(width 0.2)
-		(layer "B.Cu")
-		(net 1)
-	)
-	(segment
-		(start 485.525 164.25)
-		(end 490.91 164.25)
-		(width 0.2)
-		(layer "B.Cu")
-		(net 1)
 	)
 	(segment
@@
 	)
 	(segment
+		(start 485.775 153.025)
+		(end 495.75 143.05)
+		(width 0.2)
+		(layer "B.Cu")
+		(net 4)
+	)
+	(segment
 		(start 485.775 154)
 		(end 485.846 153.929)
@@
 	)
 	(segment
+		(start 485.775 154)
+		(end 485.775 153.025)
+		(width 0.2)
+		(layer "B.Cu")
+		(net 4)
+	)
+	(segment
 		(start 483.725 154)
 		(end 481.5 154)
@@
 	)
 	(segment
+		(start 485.525 155.815)
+		(end 495.75 145.59)
+		(width 0.2)
+		(layer "B.Cu")
+		(net 7)
+	)
+	(segment
+		(start 485.525 156.25)
+		(end 485.525 155.815)
+		(width 0.2)
+		(layer "B.Cu")
+		(net 7)
+	)
+	(segment
 		(start 458.601 163.601)
 		(end 480.279 163.601)
@@
 	)
 	(segment
-		(start 485.796 158.771)
-		(end 493.849 158.771)
-		(width 0.2)
-		(layer "B.Cu")
-		(net 8)
-	)
-	(segment
-		(start 493.849 158.771)
-		(end 495 157.62)
-		(width 0.2)
-		(layer "B.Cu")
-		(net 8)
-	)
-	(segment
 		(start 485.525 158.5)
 		(end 485.796 158.771)
@@
 		(net 11)
 	)
-	(segment
-		(start 485.55 160.75)
-		(end 491.87 160.75)
-		(width 0.2)
-		(layer "B.Cu")
-		(net 11)
-	)
-	(segment
-		(start 491.87 160.75)
-		(end 492.46 160.16)
-		(width 0.2)
-		(layer "B.Cu")
-		(net 11)
-	)

Commit message: ready for manufacturing
Routing:
- net MUX3: track 52.3 -> 66.9 mm, vias 0 -> 1
- net +3V3: track 962.5 -> 973.5 mm, vias 1 -> 2
- net MUX4: track 52.0 -> 55.4 mm, vias 0 -> 1
Changed lines of the file:
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@@
+	)
+	(segment
+		(start 475.3035 156.4625)
+		(end 474.01 156.4625)
+		(width 0.2)
+		(layer "F.Cu")
+		(net 1)
 	)
 	(segment
@@
 	)
 	(segment
+		(start 487 164.25)
+		(end 494 164.25)
+		(width 0.2)
+		(layer "F.Cu")
+		(net 1)
+	)
+	(segment
 		(start 320 173.9625)
 		(end 321 173.9625)
@@
 	)
 	(segment
-		(start 475.3035 156.4625)
-		(end 477.25 158.409)
-		(width 0.2)
-		(layer "F.Cu")
-		(net 1)
-	)
-	(segment
 		(start 120 123)
 		(end 121.75 121.25)
@@
 	)
 	(segment
-		(start 474.01 156.4625)
-		(end 475.3035 156.4625)
-		(width 0.2)
-		(layer "F.Cu")
-		(net 1)
-	)
-	(segment
 		(start 321 173.9625)
 		(end 320.47634 173.9625)
@@
 	)
 	(segment
+		(start 494 164.25)
+		(end 495.75 162.5)
+		(width 0.2)
+		(layer "F.Cu")
+		(net 1)
+	)
+	(segment
 		(start 494.3125 161.25)
 		(end 494.3125 161.1875)
@@
 	)
 	(segment
+		(start 479.83192 160.99092)
+		(end 475.3035 156.4625)
+		(width 0.2)
+		(layer "F.Cu")
+		(net 1)
+	)
+	(segment
 		(start 370 173.9625)
 		(end 368.5 175.4625)
@@
 		(net 1)
 	)
-	(via
-		(at 477.25 158.409)
-		(size 0.6)
-		(drill 0.3)
-		(layers "F.Cu" "B.Cu")
-		(net 1)
-	)
-	(segment
-		(start 477.25 160.08616)
-		(end 480.41284 163.249)
+	(segment
+		(start 479.83192 162.66808)
+		(end 479.83192 160.99092)
+		(width 0.2)
+		(layer "F.Cu")
+		(net 1)
+	)
+	(via
+		(at 487 164.25)
+		(size 0.6)
+		(drill 0.3)
+		(layers "F.Cu" "B.Cu")
+		(net 1)
+	)
+	(via
+		(at 479.83192 162.66808)
+		(size 0.6)
+		(drill 0.3)
+		(layers "F.Cu" "B.Cu")
+		(net 1)
+	)
+	(segment
+		(start 484.524 163.249)
+		(end 485.525 164.25)
+		(width 0.2)
+		(layer "B.Cu")
+		(net 1)
+	)
+	(segment
+		(start 485.525 164.25)
+		(end 487 164.25)
 		(width 0.2)
 		(layer "B.Cu")
@@
 	)
 	(segment
-		(start 477.25 158.409)
-		(end 477.25 160.08616)
-		(width 0.2)
-		(layer "B.Cu")
-		(net 1)
-	)
-	(segment
-		(start 484.524 163.249)
-		(end 485.525 164.25)
+		(start 479.83192 162.66808)
+		(end 480.41284 163.249)
 		(width 0.2)
 		(layer "B.Cu")
@@
 		(net 8)
 	)
+	(via
+		(at 487.065 156.815)
+		(size 0.6)
+		(drill 0.3)
+		(layers "F.Cu" "B.Cu")
+		(net 8)
+	)
+	(segment
+		(start 487.065 156.96)
+		(end 487.065 156.815)
+		(width 0.2)
+		(layer "B.Cu")
+		(net 8)
+	)
+	(segment
+		(start 487.065 156.815)
+		(end 495.75 148.13)
+		(width 0.2)
+		(layer "B.Cu")
+		(net 8)
+	)
+	(segment
+		(start 485.525 158.5)
+		(end 487.065 156.96)
+		(width 0.2)
+		(layer "B.Cu")
+		(net 8)
+	)
 	(segment
 		(start 485.525 158.5)
@@
 	(segment
 		(start 480.998 164.002)
+		(end 487 158)
+		(width 0.2)
+		(layer "F.Cu")
+		(net 11)
+	)
+	(segment
+		(start 487 158)
 		(end 494.33 150.67)
 		(width 0.2)
@@
 		(net 11)
 	)
+	(via
+		(at 487 158)
+		(size 0.6)
+		(drill 0.3)
+		(layers "F.Cu" "B.Cu")
+		(net 11)
+	)
+	(segment
+		(start 487 159.3)
+		(end 487 158)
+		(width 0.2)
+		(layer "B.Cu")
+		(net 11)
+	)
+	(segment
+		(start 485.55 160.75)
+		(end 487 159.3)
+		(width 0.2)
+		(layer "B.Cu")
+		(net 11)
+	)
