File: kicad/projects/chessboard_5cm/BRAIN_V2/BRAIN_V2.kicad_pcb (KiCad board)
At the start: 4 copper layers, 75 x 70 mm, 67 parts, among them J1 Conn_ARM_JTAG_SWD_10, J2 UART, J3 USB_C_Receptacle_USB2.0_16P, J4 Conn_02x03_Odd_Even, J5 I2C, J6 Conn_02x11_Odd_Even, J7 Conn_02x04_Odd_Even, J9 USB_C_Receptacle_USB2.0_16P, Q1 BC847, SW1 TL3342F450QG, U1 24LC512, U3 AP2112K-3.3, U4 AP2112K-3.3, U73 STM32L433CCTx

Commit message: two rows optimized
Routing:
- net SENSORS_REV1: track 87.2 -> 0.00 mm, vias 2 -> 0
- net +3V3: track 75.2 -> 0.00 mm, vias 21 -> 0
- net SENSORS_HW_ID1: track 73.3 -> 0.00 mm, vias 2 -> 0
- net SENSORS_REV0: track 73.2 -> 0.00 mm, vias 1 -> 0
- net SENSORS_HW_ID2: track 72.3 -> 0.00 mm, vias 1 -> 0
- net SENSORS_HW_ID0: track 67.0 -> 0.00 mm, vias 2 -> 0
- net MUX1: track 60.8 -> 0.00 mm
- net 5V_IN: track 60.5 -> 0.00 mm, vias 26 -> 0
- net MUX3: track 57.3 -> 0.00 mm
- net MUX2: track 55.5 -> 0.00 mm
- net NRF24_IRQ: track 53.5 -> 0.00 mm
- net NRF24_MOSI: track 52.6 -> 0.00 mm
- net GND: track 52.2 -> 0.00 mm, vias 124 -> 0
- net FBK_3V3_SENSORS: track 51.6 -> 0.00 mm
- net MUX4: track 51.2 -> 0.00 mm
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Other:
- board size 75 x 70 mm -> 75 x 300 mm

Commit message: interconnect 5cm finished. brain v2 with changes pending
Parts:
- removed R18, R19, R28, R29, R30: 10k, Resistor_SMD:R_0805_2012Metric_Pad1.20x1.40mm_HandSolder
- removed R31: 47k, Resistor_SMD:R_0805_2012Metric_Pad1.20x1.40mm_HandSolder
- added J10: Conn_01x08, Connector_PinSocket_2.54mm:PinSocket_1x08_P2.54mm_Horizontal, F.Cu at (110.5, 220.0)
- added J11: Conn_01x08, Connector_PinSocket_2.54mm:PinSocket_1x08_P2.54mm_Horizontal, F.Cu at (110.5, 120.0)
- added J8: Conn_01x08, Connector_PinSocket_2.54mm:PinSocket_1x08_P2.54mm_Horizontal, F.Cu at (110.5, 320.0)
- J4: value Conn_02x03_Odd_Even -> Conn_02x06_Odd_Even; footprint Connector_PinHeader_2.54mm:PinHeader_2x03_P2.54mm_Vertical_SMD -> Connector_PinSocket_2.54mm:PinSocket_2x06_P2.54mm_Vertical_SMD
- J6: value Conn_02x11_Odd_Even -> Conn_01x08; footprint Connector_PinHeader_2.54mm:PinHeader_2x11_P2.54mm_Horizontal -> Connector_PinSocket_2.54mm:PinSocket_1x08_P2.54mm_Horizontal
- R26, R27: moved to B.Cu
- moved R10 386.9 mm to (133.2, 496.2), turned to -90 degrees
- moved J3 383.8 mm to (131.9, 496.2), turned to 0 degrees
- moved R9 383.1 mm to (130.2, 496.2), turned to -90 degrees
- moved R17 372.0 mm to (120.2, 496.2), turned to -90 degrees
- moved D2 371.9 mm to (138.6, 478.6), turned to 0 degrees
- moved J9 369.9 mm to (118.2, 496.2), turned to 0 degrees
- moved SW1 369.0 mm to (144.0, 461.8), turned to 180 degrees
- moved D10 368.8 mm to (124.7, 488.5), turned to 90 degrees
- moved R14 367.9 mm to (138.4, 461.9), turned to 90 degrees
- moved R16 367.8 mm to (116.0, 496.2), turned to -90 degrees
- moved D6 367.8 mm to (141.5, 437.9)
- moved D8 367.8 mm to (143.8, 437.9)
- moved D9 367.8 mm to (146.2, 437.9)
- moved R11 367.8 mm to (141.4, 441.9)
- moved R12 367.8 mm to (143.8, 441.9)
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Connections:
- J6 pad 1: GND -> 3V3_OUT
- J6 pad 2: SIG1 -> GND
- J6 pad 3: SENSORS_REV0 -> MUX4
- J6 pad 4: SENSORS_REV1 -> MUX3
- J6 pad 5: SENSORS_HW_ID0 -> MUX2
- J6 pad 6: SENSORS_HW_ID1 -> MUX1
- J6 pad 7: 3V3_OUT -> GND
- J6 pad 8: SENSORS_HW_ID2 -> SIG1
- U73 pad 10: FBK_3V3_SENSORS -> unconnected-(U73-PA0-Pad10)
- U73 pad 2: MUX1 -> MUX4
- U73 pad 26: SENSORS_HW_ID0 -> EXPANSION4
- U73 pad 27: SENSORS_HW_ID1 -> EXPANSION3
- U73 pad 28: SENSORS_HW_ID2 -> EXPANSION2
- U73 pad 3: MUX2 -> MUX3
- U73 pad 4: MUX3 -> MUX2
- U73 pad 44: SENSORS_REV1 -> unconnected-(U73-PH3-Pad44)
- U73 pad 5: MUX4 -> MUX1
- U73 pad 6: SENSORS_REV0 -> unconnected-(U73-PH1-Pad6)
Routing:
- net MUX3: track 0.00 -> 365.1 mm, vias 0 -> 1
- net MUX2: track 0.00 -> 361.3 mm, vias 0 -> 1
- net MUX4: track 0.00 -> 357.9 mm, vias 0 -> 1
- net MUX1: track 0.00 -> 347.9 mm, vias 0 -> 1
- net SIG4: track 0.00 -> 278.3 mm
- net SIG3: track 0.00 -> 182.5 mm
- net SIG2: track 0.00 -> 87.0 mm
- net BUZZER_PWM: track 0.00 -> 67.4 mm
- net USB_P: track 0.00 -> 62.7 mm
- net USB_N: track 0.00 -> 60.8 mm
- net NRST: track 0.00 -> 46.0 mm, vias 0 -> 2
- net 3V3_OUT_EN: track 0.00 -> 45.4 mm, vias 0 -> 2
- net NRF24_CE: track 0.00 -> 41.3 mm
- net NRF24_CSN: track 0.00 -> 41.1 mm
- net NRF24_SCK: track 0.00 -> 37.1 mm
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Other:
- board size 75 x 300 mm -> 50 x 400 mm

Commit message: brain completed
Parts:
- removed J10, J11: Conn_01x08, Connector_PinSocket_2.54mm:PinSocket_1x08_P2.54mm_Horizontal
- added C2: 100nF, Capacitor_SMD:C_0805_2012Metric_Pad1.18x1.45mm_HandSolder, F.Cu at (111.0, 89.2)
- added C3: 100nF, Capacitor_SMD:C_0805_2012Metric_Pad1.18x1.45mm_HandSolder, F.Cu at (111.0, 96.0)
- added R18: 10k, Resistor_SMD:R_0805_2012Metric_Pad1.20x1.40mm_HandSolder, F.Cu at (111.0, 91.5)
- added R19: 10k, Resistor_SMD:R_0805_2012Metric_Pad1.20x1.40mm_HandSolder, F.Cu at (111.0, 93.8)
- added R24: 10k, Resistor_SMD:R_0805_2012Metric_Pad1.20x1.40mm_HandSolder, F.Cu at (119.2, 99.5)
- added SW2: TL3342F450QG, Button_Switch_SMD:SW_SPST_TL3342, F.Cu at (104.6, 85.4)
- added SW3: TL3342F450QG, Button_Switch_SMD:SW_SPST_TL3342, F.Cu at (104.5, 91.8)
- J6: value Conn_01x08 -> HCTL PM254-1-13-W-8.5; footprint Connector_PinSocket_2.54mm:PinSocket_1x08_P2.54mm_Horizontal -> Connector_PinSocket_2.54mm:PinSocket_1x13_P2.54mm_Horizontal
- J8: value Conn_01x08 -> Conn_01x02; footprint Connector_PinSocket_2.54mm:PinSocket_1x08_P2.54mm_Horizontal -> Connector_PinHeader_2.54mm:PinHeader_1x02_P2.54mm_Vertical
- moved D1 366.7 mm to (91.8, 78.6)
- moved D3 366.7 mm to (87.3, 78.6)
- moved R7 366.7 mm to (90.8, 81.6)
- moved R8 366.7 mm to (88.2, 81.6)
- moved D2 337.7 mm to (104.5, 142.6)
- moved U1 334.7 mm to (113.9, 84.9)
- moved C1 334.1 mm to (98.8, 111.6)
- moved C12 334.1 mm to (97.5, 148.1)
- moved C13 334.1 mm to (83.8, 148.1)
- moved C14 334.1 mm to (93.5, 141.1)
- moved C15 334.1 mm to (83.8, 141.1)
- moved C16 334.1 mm to (113.4, 124.5)
- moved C4 334.1 mm to (98.8, 109.4)
- moved C5 334.1 mm to (111.0, 100.5)
- moved C6 334.1 mm to (110.2, 111.8)
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Connections:
- J6 pad 1: 3V3_OUT -> GND
- J6 pad 2: GND -> 3V3_OUT
- J6 pad 3: MUX4 -> GND
- J6 pad 4: MUX3 -> SIG1
- J6 pad 5: MUX2 -> SIG2
- J6 pad 6: MUX1 -> SIG3
- J6 pad 7: GND -> SIG4
- J6 pad 8: SIG1 -> GND
- J8 pad 1: 3V3_OUT -> JUMPER
- R3 pad 1: SIG4 -> SIG1
- R4 pad 1: SIG3 -> SIG2
- R5 pad 1: SIG2 -> SIG3
- R6 pad 1: SIG1 -> SIG4
- U73 pad 10: unconnected-(U73-PA0-Pad10) -> SW_USER1
- U73 pad 44: unconnected-(U73-PH3-Pad44) -> JUMPER
- U73 pad 6: unconnected-(U73-PH1-Pad6) -> SW_USER2
Routing:
- net MUX3: track 365.1 -> 28.0 mm
- net MUX2: track 361.3 -> 26.2 mm
- net MUX4: track 357.9 -> 29.7 mm
- net MUX1: track 347.9 -> 24.5 mm
- net SIG4: track 278.3 -> 9.25 mm
- net SIG3: track 182.5 -> 10.1 mm
- net GND: track 0.00 -> 77.1 mm, vias 5 -> 128
- net SIG2: track 87.0 -> 10.9 mm
- net +3V3: track 36.9 -> 91.3 mm, vias 7 -> 29
- net 5V_IN: track 2.58 -> 38.9 mm, vias 2 -> 12
- net SW_USER1: track 0.00 -> 28.1 mm
- net BUZZER_PWM: track 67.4 -> 41.0 mm, vias 0 -> 2
- net SW_USER2: track 0.00 -> 18.1 mm
- net JUMPER: track 0.00 -> 17.6 mm, vias 0 -> 2
- net Net-(D10-A2): track 0.00 -> 16.8 mm, vias 0 -> 4
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Other:
- board size 50 x 400 mm -> 50 x 92 mm

Commit message: brain changes. all components at top and started to change into basic comps
Parts:
- R10, R16, R17, R20, R21, R22, R23, R26, R27, R9: moved to F.Cu
- moved R27 20.8 mm to (85.2, 85.0)
- moved R26 18.9 mm to (88.2, 84.0), turned to 90 degrees
- moved R22 14.4 mm to (109.5, 122.8), turned to 180 degrees
- moved R23 14.1 mm to (109.5, 125.0), turned to 0 degrees
- moved R9 9.39 mm to (105.8, 153.8), turned to 90 degrees
- moved R20 8.26 mm to (109.5, 118.2), turned to 180 degrees
- moved R16 8.12 mm to (93.0, 155.2), turned to 90 degrees
- moved R17 7.87 mm to (95.2, 155.2), turned to 90 degrees
- moved R21 7.76 mm to (109.5, 120.5), turned to 0 degrees
- moved R10 6.85 mm to (110.0, 156.5), turned to 0 degrees
- moved C16 5.43 mm to (113.2, 130.0), turned to 90 degrees
- moved R14 2.67 mm to (111.0, 130.0)
- moved R7 1.55 mm to (90.7, 80.1)
- moved R8 1.55 mm to (88.2, 80.1)
- moved D1 1.55 mm to (91.7, 77.0)
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Routing:
- net FBK_3V3_BRAIN: track 14.8 -> 37.3 mm, vias 1 -> 2
- net HWREV0: track 10.8 -> 22.3 mm, vias 1 -> 2
- net GND: track 77.1 -> 71.6 mm, vias 128 -> 124
- net HWREV1: track 7.14 -> 11.8 mm, vias 1 -> 2
- net +3V3: track 91.3 -> 86.9 mm
- net Net-(J3-CC1): track 2.98 -> 4.66 mm, vias 1 -> 0
- net NRST: track 46.0 -> 46.6 mm
- net Net-(J9-CC1): track 3.13 -> 3.57 mm, vias 1 -> 0
- net Net-(J9-CC2): track 2.88 -> 3.26 mm, vias 1 -> 0
- net 3V3_OUT: track 10.9 -> 11.2 mm, vias 5 -> 4
- net Net-(J3-CC2): track 2.92 -> 3.01 mm, vias 1 -> 0
